Commit message: update drive

File: description/ros2_control/diffbot.ros2_control.xacro (robot description, xacro)
@@ -5,25 +5,50 @@
       <hardware>
         <plugin>diffdrive_arduino/DiffDriveArduinoHardware</plugin>
-        <param name="left_wheel_name">left_wheel_joint</param>
-        <param name="right_wheel_name">right_wheel_joint</param>
+        <param name="left_wheel_names">left_front_wheel_joint, left_rear_wheel_joint</param>
+        <param name="right_wheel_names">right_front_wheel_joint, right_rear_wheel_joint</param>
         <param name="loop_rate">30</param>
-        <param name="device">/dev/serial/by-path/platform-fd500000.pcie-pci-0000:01:00.0-usb-0:1.3:1.0-port0</param>
-        <param name="baud_rate">57600</param>
+        <param name="device">/dev/esp32_motor</param>
+        <param name="baud_rate">115200</param>
         <param name="timeout_ms">1000</param>
-        <param name="enc_counts_per_rev">3436</param>
-        <param name="pid_p">20</param>
-        <param name="pid_d">12</param>
+        <param name="enc_counts_per_rev">1425</param>
+        <param name="wheel_radius">0.0722</param>
+        <param name="pid_p">2</param>
+        <param name="pid_d">1</param>
         <param name="pid_i">0</param>
         <param name="pid_o">50</param>
       </hardware>
-      <joint name="${prefix}left_wheel_joint">
-        <command_interface name="velocity"/>
-        <state_interface name="position"/>
-        <state_interface name="velocity"/>
+      <!-- Left wheels -->
+      <joint name="left_front_wheel_joint">
+          <command_interface name="velocity">
+              <param name="min">-10</param>
+              <param name="max">10</param>
+          </command_interface>
+          <state_interface name="position"/>
+          <state_interface name="velocity"/>
       </joint>
-      <joint name="${prefix}right_wheel_joint">
-        <command_interface name="velocity"/>
-        <state_interface name="position"/>
-        <state_interface name="velocity"/>
+      <joint name="left_rear_wheel_joint">
+          <command_interface name="velocity">
+              <param name="min">-10</param>
+              <param name="max">10</param>
+          </command_interface>
+          <state_interface name="position"/>
+          <state_interface name="velocity"/>
+      </joint>
+      <!-- Right wheels -->
+      <joint name="right_front_wheel_joint">
+          <command_interface name="velocity">
+              <param name="min">-10</param>
+              <param name="max">10</param>
+          </command_interface>
+          <state_interface name="position"/>
+          <state_interface name="velocity"/>
+      </joint>
+      <joint name="right_rear_wheel_joint">
+          <command_interface name="velocity">
+              <param name="min">-10</param>
+              <param name="max">10</param>
+          </command_interface>
+          <state_interface name="position"/>
+          <state_interface name="velocity"/>
       </joint>
     </ros2_control>
